Commit message: update urdf visual and LF

File: src/turtlebot5/urdf/mobile_base.xacro (robot description, xacro)
@@ -11,4 +11,8 @@
 <xacro:property name="lidar_r" value="0.025" />
 <xacro:property name="lidar_l" value="0.0215" />
+<xacro:property name="r200_cam_rgb_px" value="0.005"/>
+<xacro:property name="r200_cam_rgb_py" value="0"/>
+<xacro:property name="r200_cam_rgb_pz" value="0.013"/>
+<xacro:property name="r200_cam_depth_offset" value="0.01"/>
 <link name="base_footprint">
 </link>
@@ -151,10 +155,10 @@
 </link>
 <link name="camera_link_2">
-    <visual>
-        <origin xyz="0 0 0" rpy="1.57 0 1.57"/>
+    <!-- <visual>
+        <origin xyz="0 0 0" rpy="0 0 0"/>
         <geometry>
             <box size="0.025 0.025 0.025"/>
         </geometry>
-    </visual>
+    </visual> -->
     <collision>
         <origin xyz="0 0 0" rpy="0 0 0"/>
@@ -184,5 +188,5 @@
     <child link="platform_lift_link"/>
     <axis xyz="0 0 1"/> <!-- Movement along the Z-axis -->
-     <limit lower="0.0" upper="${(base_hight * 0.87)}" effort="50" velocity="1.0"/> <!-- Motion range and limits -->
+     <limit lower="0.04" upper="${(base_hight * 0.87)}" effort="2500" velocity="1.0"/> <!-- Motion range and limits -->
 </joint>
 <joint name="base_lidar_joint" type="fixed">
@@ -216,10 +220,34 @@
   <parent link="base_link"/>
   <child link="camera_link"/>
-  <origin xyz="${(base_length/2) + 0.009} 0 0.094" rpy="0 0 0"/>
-</joint>
+  <origin xyz="${(base_length/2) + 0.009} 0 ${0.094 + 0.05209 - (base_hight/2.0)}" rpy="0 0 0"/>
+</joint>
+<joint name="camera_rgb_joint" type="fixed">
+  <origin xyz="0 0 ${r200_cam_rgb_pz}" rpy="0 1.05 0"/>
+  <parent link="camera_link"/>
+  <child link="camera_rgb_frame"/>
+</joint>
+<link name="camera_rgb_frame"/>
+<joint name="camera_rgb_optical_joint" type="fixed">
+  <origin xyz="0 0 0" rpy="-1.57 0 -1.57"/>
+  <parent link="camera_rgb_frame"/>
+  <child link="camera_rgb_optical_frame"/>
+</joint>
+<link name="camera_rgb_optical_frame"/>
+<joint name="camera_depth_joint" type="fixed">
+  <origin xyz="${r200_cam_rgb_px} ${r200_cam_rgb_py + r200_cam_depth_offset} ${r200_cam_rgb_pz}" rpy="0 0 0"/>
+  <parent link="camera_link"/>
+  <child link="camera_depth_frame"/>
+</joint>
+<link name="camera_depth_frame"/>
+<joint name="camera_depth_optical_joint" type="fixed">
+  <origin xyz="0 0 0" rpy="-1.57 0 -1.57"/>
+  <parent link="camera_depth_frame"/>
+  <child link="camera_depth_optical_frame"/>
+</joint>
+<link name="camera_depth_optical_frame"/>
 <joint name="camera_joint_2" type="fixed">
   <parent link="base_link"/>
   <child link="camera_link_2"/>
-  <origin xyz="${(base_length/2) + 0.009} 0 0.05" rpy="0 1.05 0"/> <!-- Adjusted rpy to face the ground -->
+  <origin xyz="${(base_length/2) + 0.009} ${r200_cam_rgb_py} 0.098" rpy="0 0.5 0"/> <!-- Adjusted rpy to face the ground -->
 </joint>
 </robot>

File: src/turtlebot5/urdf/mobile_base_gazebo.xacro (robot description, xacro)
@@ -23,5 +23,5 @@
 </gazebo>
 <!-- camera test 2-->
-<gazebo reference="camera_link">
+<gazebo reference="camera_rgb_frame">
   <sensor type="depth" name="realsense_R200">
     <always_on>true</always_on>
@@ -40,5 +40,5 @@
         </clip>
     </camera>
-    <plugin name="camera_controller" filename="libgazebo_ros_openni_kinect.so">
+    <plugin name="camera_controller" filename="libgazebo_ros_camera.so">
       <baseline>0.2</baseline>
       <alwaysOn>true</alwaysOn>
@@ -68,4 +68,5 @@
 <gazebo reference="camera_link_2">
   <sensor name="camera_sensor_2" type="camera">
+    <visualize>$(arg camera_visual)</visualize>
     <update_rate>30</update_rate>
     <camera>
@@ -114,5 +115,5 @@
       <range>
         <min>0.120</min>
-        <max>3.5</max>
+        <max>10</max>
         <resolution>0.015</resolution>
       </range>

Commit message: lift system

File: src/turtlebot5/urdf/mobile_base.xacro (robot description, xacro)
@@ -58,5 +58,5 @@
   </visual>
   <collision>
-      <origin xyz="0.0 0.0 0.0" rpy="${pi / 2.0} 0.0 0.0"/>
+      <origin xyz="0.0 0.0 ${0.18/2}" rpy="0.0 0.0 0.0"/>
     <geometry>
         <cylinder radius="${0.05}" length="${0.18}"/>
@@ -64,5 +64,5 @@
     <material name="red"/>
   </collision>
-  <xacro:cylinder_inertia m="1.0" r="${2*wheel_r}" h="${2*wheel_length}" xyz="0.0 0.0 0.0" rpy="${pi / 2.0} 0.0 0.0" />
+  <xacro:cylinder_inertia m="1.0" r="${2*wheel_r}" h="${2*wheel_length}" xyz="0.0 0.0 ${0.18/2}" rpy="0.0 0.0 0.0" />
 </link>
 <link name="lidar_link">
