Commit message: visual

File: src/turtlebot5/urdf/turtlebot5.xacro (robot description, xacro)
@@ -249,5 +249,5 @@
   <parent link="base_link"/>
   <child link="camera_link_2"/>
-  <origin xyz="${(base_length/2) + 0.009} ${r200_cam_rgb_py} 0.098" rpy="0 0.5 0"/> <!-- Adjusted rpy to face the ground -->
+  <origin xyz="${(base_length/2) + 0.09} ${r200_cam_rgb_py} 0.098" rpy="0 0.5 0"/> <!-- Adjusted rpy to face the ground -->
 </joint>
 </robot>
