Commit message: gmapping

File: src/turtlebot5/urdf/turtlebot5.gazebo.xacro (robot description, xacro)
@@ -6,8 +6,8 @@
   <material>Gazebo/Blue</material>
 </gazebo>
-<gazebo reference="left_wheel_link">
+<gazebo reference="wheel_left_link">
   <material>Gazebo/Grey</material>
 </gazebo>
-<gazebo reference="right_wheel_link">
+<gazebo reference="wheel_right_link">
   <material>Gazebo/Grey</material>
 </gazebo>
@@ -98,5 +98,5 @@
   </sensor>
 </gazebo>
-<gazebo reference="lidar_link">
+<gazebo reference="base_scan">
   <material>Gazebo/FlatBlack</material>
   <sensor type="ray" name="lds_lfcd_sensor">
@@ -131,5 +131,5 @@
 </gazebo>
 <gazebo>
-  <plugin name="differential_drive_controller" filename="libgazebo_ros_diff_drive.so">
+  <plugin name="turtlebot5_controller" filename="libgazebo_ros_diff_drive.so">
     <legacyMode>true</legacyMode>
     <rosDebugLevel>Debug</rosDebugLevel>
@@ -140,6 +140,6 @@
     <alwaysOn>true</alwaysOn>
     <updateRate>100.0</updateRate>
-    <leftJoint>left_wheel_joint</leftJoint>
-    <rightJoint>right_wheel_joint</rightJoint>
+    <leftJoint>wheel_left_joint</leftJoint>
+    <rightJoint>wheel_right_joint</rightJoint>
     <wheelSeparation>${base_width}</wheelSeparation>
     <wheelDiameter>${wheel_r * 2}</wheelDiameter>
@@ -160,6 +160,6 @@
 </gazebo>
 <!-- Transmissions for ROS Control -->
-<xacro:transmission_block joint_name="left_wheel_joint"/>
-<xacro:transmission_block joint_name="right_wheel_joint"/>
+<xacro:transmission_block joint_name="wheel_left_joint"/>
+<xacro:transmission_block joint_name="wheel_right_joint"/>
 <transmission name="prismatic_trans">
   <type>transmission_interface/SimpleTransmission</type>
@@ -173,6 +173,7 @@
 <!-- ROS control plugin -->
 <gazebo>
-  <plugin name="gazebo_ros_control" filename="libgazebo_ros_control.so">
-  </plugin>
+    <plugin name="gazebo_ros_control" filename="libgazebo_ros_control.so">
+        <robotNamespace>/</robotNamespace>
+    </plugin>
 </gazebo>
 </robot>

File: src/turtlebot5/urdf/turtlebot5.xacro (robot description, xacro)
@@ -33,4 +33,21 @@
   <xacro:box_inertia m="5.0" l="${2*base_length}" w="${2*base_width}" h="${2*base_hight}" xyz="0.0 0.0 ${base_hight/2.0}" rpy="0.0 0.0 0.0"/>
 </link>
+<link name="platform_lift_link">
+  <visual>
+    <origin xyz="0.0 0.0 0.0" rpy="0 0.0 0.0"/>
+    <geometry>
+        <mesh filename="package://turtlebot5/meshes/inner.stl"/>
+    </geometry>
+    <material name="grey"/>
+  </visual>
+  <!-- <collision>
+      <origin xyz="0.0 0.0 ${0.18/2}" rpy="0.0 0.0 0.0"/>
+    <geometry>
+        <cylinder radius="${0.05}" length="${0.18}"/>
+    </geometry>
+    <material name="red"/>
+  </collision>    -->
+  <xacro:cylinder_inertia m="1.0" r="${2*wheel_r}" h="${2*wheel_length}" xyz="0.0 0.0 ${0.18/2}" rpy="0.0 0.0 0.0" />
+</link>
 <link name="platform_link">
   <visual>
@@ -49,22 +66,5 @@
   <xacro:box_inertia m="5.0" l="0.35" w="0.22" h="0.026" xyz="0.0 0.0 0" rpy="0.0 0.0 0.0"/>
 </link>
-<link name="platform_lift_link">
-  <visual>
-    <origin xyz="0.0 0.0 0.0" rpy="0 0.0 0.0"/>
-    <geometry>
-        <mesh filename="package://turtlebot5/meshes/inner.stl"/>
-    </geometry>
-    <material name="grey"/>
-  </visual>
-  <collision>
-      <origin xyz="0.0 0.0 ${0.18/2}" rpy="0.0 0.0 0.0"/>
-    <geometry>
-        <cylinder radius="${0.05}" length="${0.18}"/>
-    </geometry>
-    <material name="red"/>
-  </collision>
-  <xacro:cylinder_inertia m="1.0" r="${2*wheel_r}" h="${2*wheel_length}" xyz="0.0 0.0 ${0.18/2}" rpy="0.0 0.0 0.0" />
-</link>
-<link name="lidar_link">
+<link name="base_scan">
     <visual name="">
         <origin xyz="0.0 0.0 0.0" rpy="0.0 0.0 0.0"/>
@@ -81,5 +81,5 @@
     </collision>
 </link>
-<link name="left_wheel_link">
+<link name="wheel_left_link">
   <visual>
     <origin xyz="0.0 0.0 0.0" rpy="${pi / 2.0} 0.0 0.0"/>
@@ -97,5 +97,5 @@
   <xacro:cylinder_inertia m="1.0" r="${2*wheel_r}" h="${2*wheel_length}" xyz="0.0 0.0 0.0" rpy="${pi / 2.0} 0.0 0.0" />
 </link>
-<link name="right_wheel_link">
+<link name="wheel_right_link">
   <visual>
       <origin xyz="0.0 0.0 0.0" rpy="${pi / 2.0} 0.0 0.0"/>
@@ -188,20 +188,20 @@
     <child link="platform_lift_link"/>
     <axis xyz="0 0 1"/> <!-- Movement along the Z-axis -->
-     <limit lower="0.04" upper="${(base_hight * 0.87)}" effort="2500" velocity="1.0"/> <!-- Motion range and limits -->
+    <limit lower="0.04" upper="${(base_hight * 0.87)}" effort="2500" velocity="1.0"/> <!-- Motion range and limits -->
 </joint>
 <joint name="base_lidar_joint" type="fixed">
     <parent link="base_link"/>
-    <child link="lidar_link"/>
+    <child link="base_scan"/>
     <origin xyz="${(base_length / 2)- lidar_r} 0.0 ${(base_hight + lidar_l / 2) - 0.005}" rpy="0.0 0.0 0.0"/>
 </joint>
-<joint name="left_wheel_joint" type="continuous">
-    <parent link="base_link"/>
-    <child link="left_wheel_link"/>
+<joint name="wheel_left_joint" type="continuous">
+    <parent link="base_link"/>
+    <child link="wheel_left_link"/>
     <origin xyz="0 ${(base_width + wheel_length)/2.0} 0.0" rpy="0.0 0.0 0.0"/>
     <axis xyz="0 1 0.0"/>
 </joint>
-<joint name="right_wheel_joint" type="continuous">
-    <parent link="base_link"/>
-    <child link="right_wheel_link"/>
+<joint name="wheel_right_joint" type="continuous">
+    <parent link="base_link"/>
+    <child link="wheel_right_link"/>
     <origin xyz=" 0 ${-(base_width + wheel_length)/2.0} 0.0" rpy="0.0 0.0 0.0"/>
     <axis xyz="0 1 0.0"/>

Commit message: junction system fixed

File: src/turtlebot5/urdf/turtlebot5.gazebo.xacro (robot description, xacro)
@@ -22,5 +22,5 @@
   <mu2 value="0.1"/>
 </gazebo>
-<!-- camera test 2-->
+<!-- cameras-->
 <gazebo reference="camera_rgb_frame">
   <sensor type="depth" name="realsense_R200">
@@ -98,4 +98,85 @@
   </sensor>
 </gazebo>
+<gazebo reference="camera_left">
+  <sensor type="depth" name="realsense_R200">
+    <always_on>true</always_on>
+    <visualize>$(arg camera_visual)</visualize>
+    <camera>
+        <horizontal_fov>1.3439</horizontal_fov>
+        <image>
+            <width>1920</width>
+            <height>1080</height>
+            <format>R8G8B8</format>
+        </image>
+        <depth_camera></depth_camera>
+        <clip>
+            <near>0.03</near>
+            <far>100</far>
+        </clip>
+    </camera>
+    <plugin name="camera_controller" filename="libgazebo_ros_camera.so">
+      <baseline>0.2</baseline>
+      <alwaysOn>true</alwaysOn>
+      <updateRate>30.0</updateRate>
+      <cameraName>camera_left</cameraName>
+      <imageTopicName>camera_left/image_raw</imageTopicName>
+      <cameraInfoTopicName>camera_left/camera_info</cameraInfoTopicName>
+      <frameName>camera_left</frameName>
+      <pointCloudCutoff>0.4</pointCloudCutoff>
+          <hackBaseline>0.07</hackBaseline>
+          <distortionK1>0.0</distortionK1>
+          <distortionK2>0.0</distortionK2>
+          <distortionK3>0.0</distortionK3>
+          <distortionT1>0.0</distortionT1>
+          <distortionT2>0.0</distortionT2>
+      <CxPrime>0.0</CxPrime>
+      <Cx>0.0</Cx>
+      <Cy>0.0</Cy>
+      <focalLength>0</focalLength>
+      <hackBaseline>0</hackBaseline>
+    </plugin>
+  </sensor>
+</gazebo>
+<gazebo reference="camera_right">
+  <sensor type="depth" name="realsense_R200">
+    <always_on>true</always_on>
+    <visualize>$(arg camera_visual)</visualize>
+    <camera>
+        <horizontal_fov>1.3439</horizontal_fov>
+        <image>
+            <width>1920</width>
+            <height>1080</height>
+            <format>R8G8B8</format>
+        </image>
+        <depth_camera></depth_camera>
+        <clip>
+            <near>0.03</near>
+            <far>100</far>
+        </clip>
+    </camera>
+    <plugin name="camera_controller" filename="libgazebo_ros_camera.so">
+      <baseline>0.2</baseline>
+      <alwaysOn>true</alwaysOn>
+      <updateRate>30.0</updateRate>
+      <cameraName>camera_right</cameraName>
+      <frameName>camera_right</frameName>
+      <imageTopicName>camera_right/image_raw</imageTopicName>
+      <cameraInfoTopicName>camera_right/camera_info</cameraInfoTopicName>
+      <pointCloudCutoff>0.4</pointCloudCutoff>
+          <hackBaseline>0.07</hackBaseline>
+          <distortionK1>0.0</distortionK1>
+          <distortionK2>0.0</distortionK2>
+          <distortionK3>0.0</distortionK3>
+          <distortionT1>0.0</distortionT1>
+          <distortionT2>0.0</distortionT2>
+      <CxPrime>0.0</CxPrime>
+      <Cx>0.0</Cx>
+      <Cy>0.0</Cy>
+      <focalLength>0</focalLength>
+      <hackBaseline>0</hackBaseline>
+    </plugin>
+  </sensor>
+</gazebo>
+<!--scan-->
 <gazebo reference="base_scan">
   <material>Gazebo/FlatBlack</material>

File: src/turtlebot5/urdf/turtlebot5.xacro (robot description, xacro)
@@ -8,4 +8,5 @@
 <xacro:property name="wheel_r" value="0.051" />
 <xacro:property name="wheel_length" value="0.046" />
+<xacro:property name="wheel_margin" value="0.015" />
 <!-- Lidar values  -->
 <xacro:property name="lidar_r" value="0.025" />
@@ -168,4 +169,22 @@
     </collision>
 </link>
+<link name="camera_left">
+  <visual>
+   <origin xyz="0.0 0.0 0.0" rpy="1.57 0 1.57"/>
+    <geometry>
+      <box size="0.025 0.025 0.025"/>
+    </geometry>
+    <material name="grey"/>
+  </visual>
+</link>
+<link name="camera_right">
+  <visual>
+   <origin xyz="0.0 0.0 0.0" rpy="1.57 0 1.57"/>
+    <geometry>
+      <box size="0.025 0.025 0.025"/>
+    </geometry>
+    <material name="grey"/>
+  </visual>
+</link>
 <!-- ####################################################################################################################### -->
 <!-- ####################################################################################################################### -->
@@ -198,5 +217,5 @@
     <parent link="base_link"/>
     <child link="wheel_left_link"/>
-    <origin xyz="0 ${(base_width + wheel_length)/2.0} 0.0" rpy="0.0 0.0 0.0"/>
+    <origin xyz="0 ${(base_width - wheel_length + wheel_margin)/2.0} 0.0" rpy="0.0 0.0 0.0"/>
     <axis xyz="0 1 0.0"/>
 </joint>
@@ -204,5 +223,5 @@
     <parent link="base_link"/>
     <child link="wheel_right_link"/>
-    <origin xyz=" 0 ${-(base_width + wheel_length)/2.0} 0.0" rpy="0.0 0.0 0.0"/>
+    <origin xyz=" 0 ${-(base_width - wheel_length + wheel_margin)/2.0} 0.0" rpy="0.0 0.0 0.0"/>
     <axis xyz="0 1 0.0"/>
 </joint>
@@ -249,5 +268,15 @@
   <parent link="base_link"/>
   <child link="camera_link_2"/>
-  <origin xyz="${(base_length/2) + 0.09} ${r200_cam_rgb_py} 0.098" rpy="0 0.5 0"/> <!-- Adjusted rpy to face the ground -->
+  <origin xyz="${(base_length/2) + 0.09} ${r200_cam_rgb_py + (0.098/2)} 0.098" rpy="0 0.5 0"/> <!-- Adjusted rpy to face the ground -->
+</joint>
+<joint name="camera_left_joint" type="fixed">
+  <parent link="base_link"/>
+  <child link="camera_left"/>
+  <origin xyz="0 ${(base_width)/2.0} ${0.12 + 0.05209 - (base_hight/2.0)}" rpy="0 1.05 1.5708"/> <!-- Adjusted rpy to face the ground -->
+</joint>
+<joint name="camera_right_joint" type="fixed">
+  <parent link="base_link"/>
+  <child link="camera_right"/>
+  <origin xyz="0 ${-(base_width)/2.0} ${0.12 + 0.05209 - (base_hight/2.0)}" rpy="0 1.05 -1.5708"/> <!-- Adjusted rpy to face the ground -->
 </joint>
 </robot>
